Commit message: Add world.

File: src/vehicle_description/urdf/vehicle.xacro (robot description, xacro)
@@ -4,5 +4,5 @@
   <!-- Constants for robot dimensions -->
   <xacro:property name="PI" value="3.1415926535897931"/>
-  <xacro:property name="mass" value="10" /> <!-- arbitrary value for mass -->
+  <xacro:property name="mass" value="1" /> <!-- arbitrary value for mass -->
   <xacro:property name="width" value="0.3" /> <!-- Square dimensions (widthxwidth) of vehicle body -->
   <xacro:property name="length" value="0.5" /> <!-- Link 1 -->
@@ -112,5 +112,5 @@
     <inertial>
       <origin xyz="0 ${wheel_t/2+gap} 0" rpy="${PI/2} 0 0"/>
-      <mass value="${mass}"/>
+      <mass value="${mass/10}"/>
       <inertia
 			ixx="${mass / 12.0 * (wheel_t*wheel_t*2)}" ixy="0.0" ixz="0.0"
@@ -136,5 +136,5 @@
     <inertial>
       <origin xyz="0 ${-wheel_t/2-gap} 0" rpy="${PI/2} 0 0"/>
-      <mass value="${mass}"/>
+      <mass value="${mass/10}"/>
       <inertia
 			ixx="${mass / 12.0 * (wheel_t*wheel_t*2)}" ixy="0.0" ixz="0.0"
@@ -160,5 +160,5 @@
     <inertial>
       <origin xyz="0 ${wheel_t/2+gap} 0" rpy="${PI/2} 0 0"/>
-      <mass value="${mass}"/>
+      <mass value="${mass/10}"/>
       <inertia
 			ixx="${mass / 12.0 * (wheel_t*wheel_t*2)}" ixy="0.0" ixz="0.0"
@@ -184,5 +184,5 @@
     <inertial>
       <origin xyz="0 ${-wheel_t/2-gap} 0" rpy="${PI/2} 0 0"/>
-      <mass value="${mass}"/>
+      <mass value="${mass/10}"/>
       <inertia
 			ixx="${mass / 12.0 * (wheel_t*wheel_t*2)}" ixy="0.0" ixz="0.0"
@@ -230,43 +230,3 @@
   <link name="camera_link_optical">
   </link>
-  <transmission name="tran1">
-    <type>transmission_interface/SimpleTransmission</type>
-    <joint name="joint1">
-      <hardwareInterface>hardware_interface/EffortJointInterface</hardwareInterface>
-    </joint>
-    <actuator name="motor1">
-      <hardwareInterface>hardware_interface/EffortJointInterface</hardwareInterface>
-      <mechanicalReduction>1</mechanicalReduction>
-    </actuator>
-  </transmission>
-  <transmission name="tran2">
-    <type>transmission_interface/SimpleTransmission</type>
-    <joint name="joint2">
-      <hardwareInterface>hardware_interface/EffortJointInterface</hardwareInterface>
-    </joint>
-    <actuator name="motor2">
-      <hardwareInterface>hardware_interface/EffortJointInterface</hardwareInterface>
-      <mechanicalReduction>1</mechanicalReduction>
-    </actuator>
-  </transmission>
-  <transmission name="tran3">
-    <type>transmission_interface/SimpleTransmission</type>
-    <joint name="joint2">
-      <hardwareInterface>hardware_interface/EffortJointInterface</hardwareInterface>
-    </joint>
-    <actuator name="motor3">
-      <hardwareInterface>hardware_interface/EffortJointInterface</hardwareInterface>
-      <mechanicalReduction>1</mechanicalReduction>
-    </actuator>
-  </transmission>
-  <transmission name="tran4">
-    <type>transmission_interface/SimpleTransmission</type>
-    <joint name="joint4">
-      <hardwareInterface>hardware_interface/EffortJointInterface</hardwareInterface>
-    </joint>
-    <actuator name="motor4">
-      <hardwareInterface>hardware_interface/EffortJointInterface</hardwareInterface>
-      <mechanicalReduction>1</mechanicalReduction>
-    </actuator>
-  </transmission>
 </robot>
